Commit message: Add files via upload

File: urdf/object2.urdf (robot description, URDF)
Before this commit: robot myrobot, 6 links, 5 joints
Links:
- link Box: geometry visual box size=0.8 0.4 0.4

File: urdf/robot.urdf (robot description, URDF)
Before this commit: robot myrobot, 9 links, 8 joints
Links:
- link link0: geometry collision cylinder length=2.5 radius=0.35; visual cylinder length=2.5 radius=0.35
- link link1: geometry collision cylinder length=3.5 radius=0.2; visual cylinder length=3.5 radius=0.2
- link link2: geometry collision cylinder length=3 radius=0.1; visual cylinder length=3 radius=0.1
Joints:
- joint link0_to_link1: origin xyz=0 0 2 rpy=0 0 0 -> xyz=0 0 2.5 rpy=0 0 0
- joint link1_to_link2: origin xyz=0 0 3 rpy=0 0 0 -> xyz=0 0 3.5 rpy=0 0 0
- joint sphere2_to_link2: origin xyz=0 0 2 rpy=0 0 0 -> xyz=0 0 3 rpy=0 0 0
